Commit message: New localizer added, gps sensor modified, some bug fixes

File: sgd_bringup/urdf/sgd_model.urdf (robot description, URDF)
Before this commit: robot turtlebot3_waffle, 13 links, 12 joints
Links:
- removed link caster_back_left_link
- removed link caster_back_right_link
- added link caster_link, mass 2; collision sphere radius=0.15; visual sphere radius=0.15
- added link gps_link, mass 0.1; collision box size=0.05 0.05 0.05; visual box size=0.05 0.05 0.05
- link base_link: mass 1.3729096e+00 -> 8; geometry collision box size=0.7152 0.1 0.2; visual box size=0.7152 0.1 0.2
- link base_scan: geometry collision cylinder length=0.055 radius=0.0508; visual mesh filename=package://turtlebot3_description/meshes/sensors/lds.stl scale=0.001 0.001 0.001
- link wheel_left_link: mass 2.8498940e-02 -> 2; geometry collision cylinder length=0.056 radius=0.1523; visual cylinder length=0.056 radius=0.1523
- link wheel_right_link: mass 2.8498940e-02 -> 2; geometry collision cylinder length=0.056 radius=0.1523; visual cylinder length=0.056 radius=0.1523
Joints:
- removed joint caster_back_left_joint
- removed joint caster_back_right_joint
- added joint caster_joint: type fixed, parent base_link, child caster_link, origin xyz=0.7152 0 -0.0774 rpy=0 0 0
- added joint gps_joint: type fixed, parent base_link, child gps_link, origin xyz=0.3 0 0.3 rpy=0 0 0
- joint base_joint: origin xyz=0 0 0.010 rpy=0 0 0 -> xyz=0 0 0.1524 rpy=0 0 0
- joint camera_joint: origin xyz=0.064 -0.065 0.094 rpy=0 0 0 -> xyz=0.64 -0.065 0.094 rpy=0 0 0
- joint imu_joint: origin xyz=0.0 0 0.068 rpy=0 0 0 -> xyz=0.0 0 0.3 rpy=0 0 0
- joint scan_joint: origin xyz=-0.064 0 0.122 rpy=0 0 0 -> xyz=0.6 0 0.3 rpy=0 0 0
- joint wheel_left_joint: origin xyz=0.0 0.144 0.023 rpy=-1.57 0 0 -> xyz=0 0.3493 0 rpy=-1.57 0 0
- joint wheel_right_joint: origin xyz=0.0 -0.144 0.023 rpy=-1.57 0 0 -> xyz=0 -0.3493 0 rpy=-1.57 0 0

Commit message: Implementation of Kalman Filter for localization. Logger node added.

File: sgd_bringup/urdf/sgd_model.urdf (robot description, URDF)
Before this commit: robot turtlebot3_waffle, 13 links, 12 joints
Links:
- removed link camera_depth_frame
- removed link camera_depth_optical_frame
- removed link camera_link
- removed link camera_rgb_frame
- removed link camera_rgb_optical_frame
- link imu_link: mass None -> 0.01; geometry collision box size=0.1 0.1 0.1; visual box size=0.1 0.1 0.1
Joints:
- removed joint camera_depth_joint
- removed joint camera_depth_optical_joint
- removed joint camera_joint
- removed joint camera_rgb_joint
- removed joint camera_rgb_optical_joint

Commit message: Navigation implementation, localization is not working!

File: sgd_bringup/urdf/sgd_model.urdf (robot description, URDF)
Before this commit: robot shared_guide_dog, 8 links, 7 joints
Links:
- link wheel_left_link: geometry collision cylinder length=0.056 radius=0.1082; visual cylinder length=0.056 radius=0.1082
- link wheel_right_link: geometry collision cylinder length=0.056 radius=0.1082; visual cylinder length=0.056 radius=0.1082
Joints:
- joint wheel_left_joint: origin xyz=0 0.3493 0 rpy=-1.57 0 0 -> xyz=0 0.3493 -0.05 rpy=-1.57 0 0
- joint wheel_right_joint: origin xyz=0 -0.3493 0 rpy=-1.57 0 0 -> xyz=0 -0.3493 -0.05 rpy=-1.57 0 0

Commit message: Final commit for masters thesis

File: sgd_bringup/urdf/sgd_model.urdf (robot description, URDF)
Before this commit: robot shared_guide_dog, 8 links, 7 joints
Joints:
- joint scan_joint: origin xyz=0.6 0 0.3 rpy=0 0 0 -> xyz=0.6 0 0.4 rpy=0 0 0

Commit message: AMCL integration

File: sgd_bringup/urdf/sgd_model.urdf (robot description, URDF)
Before this commit: robot shared_guide_dog, 8 links, 7 joints
Links:
- removed link base_footprint
- link caster_link: geometry collision sphere radius=0.1082; visual sphere radius=0.1082
Joints:
- removed joint base_joint
- joint scan_joint: origin xyz=0.6 0 0.4 rpy=0 0 0 -> xyz=0.6 0 0.4 rpy=3.14159 0 0

Commit message: New simulation world

File: sgd_bringup/urdf/sgd_model.urdf (robot description, URDF)
Before this commit: robot shared_guide_dog, 7 links, 6 joints
Links:
- added link base_frame, mass 8; collision box size=0.7152 0.1 0.2; visual box size=0.7152 0.5 0.2
- link base_link: mass 8 -> None; geometry 
Joints:
- added joint base_frame_joint: type fixed, parent base_link, child base_frame, origin xyz=0.0 0 0.3 rpy=0 0 0
- joint caster_joint: parent base_link -> base_frame
- joint gps_joint: parent base_link -> base_frame
- joint imu_joint: parent base_link -> base_frame
- joint scan_joint: parent base_link -> base_frame
- joint wheel_left_joint: parent base_link -> base_frame
- joint wheel_right_joint: parent base_link -> base_frame

Commit message: software version for BSVH meeting

File: sgd_bringup/urdf/sgd_model.urdf (robot description, URDF)
Before this commit: robot shared_guide_dog, 8 links, 7 joints
Joints:
- joint gps_joint: origin xyz=0.3 0 0.3 rpy=0 0 0 -> xyz=0.5 0 0.3 rpy=0 0 0

Commit message: Fixed build order, rework of most hardware drivers, deleted old packages.

File: sgd_bringup/urdf/sgd_model.urdf (robot description, URDF)
Before this commit: robot shared_guide_dog, 8 links, 7 joints
Links:
- added link uwb_link, mass 0.1; collision box size=0.05 0.05 0.05; visual box size=0.05 0.05 0.05
Joints:
- added joint uwb_joint: type fixed, parent base_frame, child uwb_link, origin xyz=0.36 0 1.13 rpy=0 0 0
- joint gps_joint: origin xyz=0.5 0 0.3 rpy=0 0 0 -> xyz=0.75 0 0.7 rpy=0 0 0
- joint imu_joint: origin xyz=0.0 0 0.3 rpy=0 0 0 -> xyz=0.4 0 0.95 rpy=0 0 0
- joint scan_joint: origin xyz=0.6 0 0.4 rpy=3.14159 0 0 -> xyz=0.85 0 0.42 rpy=3.14159 0 0

Commit message: Added a helper function for scan playback; fixed a bug in sgd_io package; added some maps

File: sgd_bringup/urdf/sgd_model.urdf (robot description, URDF)
Before this commit: robot shared_guide_dog, 9 links, 8 joints
Joints:
- joint gps_joint: origin xyz=0.75 0 0.7 rpy=0 0 0 -> xyz=0.45 0 1.1 rpy=0 0 0
